File: Migouner2.kicad_sch (KiCad schematic)
At the start: 0 parts

Commit message: Update Migouner2.kicad_pcb, Migouner2.kicad_prl, Migouner2.kicad_pro, and 4 more files
Other:
- sheet Keyboard Matrix ports: added Col10, Col11, Col12, Col13, Col14, Col15, Col16, Col17, Col18, Col2, Col3, Col4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; removed none
- sheet STM32 ports: added LED, M0, M1, M10, M11, M12, M13, M14, M15, M16, M17, M18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; removed PA14, PA15, PB3, PB4, PB5
