File: STM32.kicad_sch (KiCad schematic)
At the start: 17 parts, among them J1 USB_B_Micro, U1 STM32F072CBT6, U2 XC6206P332MR-G, U7 ZX-PZ2.54-2-5PZZ

Commit message: Update Migouner2.kicad_pcb, Migouner2.kicad_prl, Migouner2.kicad_pro, and 4 more files
Parts:
- removed U7: ZX-PZ2.54-2-5PZZ, JLClib:HDR-TH_6P-P2.54-V-M-R2-C3-S2.54-1, symbol JLClib:Header-Male-2.54_2x3
- SW1: value ~ -> Boot Switch
- renumbered U1 to X1, U2 to X2
Connections:
- net Boot: now also SW1.4 (D); no longer R1.2
- net GND: now also R1.1; no longer SW1.3 (C)
- net M0: now reaches X1.10 (PA0)
- net M18: now reaches X1.11 (PA1)
- net M19: now reaches X1.12 (PA2)
- net M20: now reaches X1.13 (PA3)
- net M21: now reaches X1.14 (PA4)
- net M22: now reaches X1.15 (PA5)
- net M23: now reaches X1.16 (PA6)
- net LED: now reaches X1.17 (PA7)
- net M17: now reaches X1.25 (PB12)
- net M16: now reaches X1.26 (PB13)
- net M15: now reaches X1.27 (PB14)
- net M14: now reaches X1.28 (PB15)
- net M13: now reaches X1.29 (PA8)
- net M12: now reaches X1.30 (PA9)
- net M11: now reaches X1.31 (PA10)
- net M10: now reaches X1.34 (PA13)
- net M4: now reaches X1.42 (PB6)
- net M3: now reaches X1.43 (PB7)
- net M2: now reaches X1.45 (PB8)
- net M1: now reaches X1.46 (PB9)
- net PA14 renamed M9
- net PA15 renamed M8
- net PB3 renamed M7
- net PB4 renamed M6
- net PB5 renamed M5
- new net: R1.2, SW1.3 (C)
Other:
- moved on the sheet: R1, SW1
