File: STM32.kicad_sch (KiCad schematic)
At the start: 17 parts, among them J1 USB_B_Micro, U1 STM32F072CBT6, U2 XC6206P332MR-G, U7 ZX-PZ2.54-2-5PZZ

Commit message: Corrected Devboard
Parts:
- removed U7: ZX-PZ2.54-2-5PZZ, JLClib:HDR-TH_6P-P2.54-V-M-R2-C3-S2.54-1, symbol JLClib:Header-Male-2.54_2x3
- added J2: Conn_01x04_Pin, Connector_PinHeader_1.27mm:PinHeader_2x02_P1.27mm_Vertical, symbol Connector_Generic:Conn_02x02_Counter_Clockwise
Connections:
- net +3.3V: now also J2.4 (Pin_4)
- net +5V: now also J2.2 (Pin_2)
- net Boot: now also SW1.4 (D), J2.3 (Pin_3); no longer R1.2
- net GND: now also R1.2, J2.1 (Pin_1); no longer SW1.3 (C)
- net at R1.1: now also SW1.3 (C); no longer SW1.4 (D)
Other:
- note added: "External Pin Headers"
- moved on the sheet: R1, SW1
