File: Migouner2.kicad_pcb (KiCad board)
At the start: 2 copper layers, 52.4 x 38.1 mm, 38 parts, among them J1 USB_B_Micro, SW2 A, SW3 S, SW4 D, SW5 W, U1 STM32F072CBT6, U2 XC6206P332MR-G, U3 A, U4 D, U5 S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

Commit message: Corrected Devboard
Parts:
- removed U7: ZX-PZ2.54-2-5PZZ, JLClib:HDR-TH_6P-P2.54-V-M-R2-C3-S2.54-1
- added J2: Conn_01x04_Pin, Connector_PinHeader_1.27mm:PinHeader_2x02_P1.27mm_Vertical, F.Cu at (166.9, 61.6)
- moved R1 5.92 mm to (174.8, 82.5), turned to 180 degrees
Connections:
- R1 pad 1: Net-(SW1-D) -> Net-(SW1-C)
- R1 pad 2: /STM32/Boot -> GND
- SW1 pad 3: GND -> Net-(SW1-C)
- SW1 pad 4: Net-(SW1-D) -> /STM32/Boot
- U1 pad 25: Net-(U1-PB12) -> unconnected-(U1-PB12-Pad25)
- U1 pad 26: Net-(U1-PB13) -> unconnected-(U1-PB13-Pad26)
- U1 pad 27: Net-(U1-PB14) -> unconnected-(U1-PB14-Pad27)
- U1 pad 28: Net-(U1-PB15) -> unconnected-(U1-PB15-Pad28)
Routing:
- net /STM32/Boot: track 3.70 -> 29.4 mm, vias 0 -> 1
- net Net-(U1-PB15): track 12.7 -> 0.00 mm, vias 1 -> 0
- net Net-(U1-PB12): track 12.6 -> 0.00 mm
- net Net-(U1-PB14): track 9.97 -> 0.00 mm, vias 1 -> 0
- net Net-(U1-PB13): track 9.95 -> 0.00 mm
- net Net-(SW1-D): track 9.47 -> 0.00 mm, vias 1 -> 0
- net GND: track 39.7 -> 34.1 mm, vias 8 -> 7
- net +3.3V: track 66.8 -> 71.8 mm
- net Net-(SW1-C): track 0.00 -> 3.17 mm, vias 0 -> 1
- net +5V: track 114.0 -> 115.3 mm
Other:
- board text added: "3.3V"
- board text added: "5V"
- board text added: "Boot0"
- board text added: "GND"
- board text removed: "GND 5V"
