File: Migouner2.kicad_pcb (KiCad board)
At the start: 2 copper layers, 52.4 x 38.1 mm, 38 parts, among them J1 USB_B_Micro, SW2 A, SW3 S, SW4 D, SW5 W, U1 STM32F072CBT6, U2 XC6206P332MR-G, U3 A, U4 D, U5 S, U6 W, U7 ZX-PZ2.54-2-5PZZ

Commit message: Update Migouner2.kicad_pcb, Migouner2.kicad_prl, Migouner2.kicad_pro, and 4 more files
Parts:
- added D10: A, JLClib:SOD-323_L1.8-W1.3-LS2.5-RD, F.Cu at (-20.3, 151.8)
- added D11: A, JLClib:SOD-323_L1.8-W1.3-LS2.5-RD, F.Cu at (-20.3, 154.4)
- added D12: A, JLClib:SOD-323_L1.8-W1.3-LS2.5-RD, F.Cu at (-20.3, 157.0)
- added D13: A, JLClib:SOD-323_L1.8-W1.3-LS2.5-RD, F.Cu at (-20.3, 159.6)
- added D14: A, JLClib:SOD-323_L1.8-W1.3-LS2.5-RD, F.Cu at (-20.3, 162.2)
- added D15: A, JLClib:SOD-323_L1.8-W1.3-LS2.5-RD, F.Cu at (-20.3, 164.9)
- added D16: A, JLClib:SOD-323_L1.8-W1.3-LS2.5-RD, F.Cu at (-15.9, 136.1)
- added D17: A, JLClib:SOD-323_L1.8-W1.3-LS2.5-RD, F.Cu at (-15.9, 138.8)
- added D18: A, JLClib:SOD-323_L1.8-W1.3-LS2.5-RD, F.Cu at (-15.9, 141.4)
- added D19: A, JLClib:SOD-323_L1.8-W1.3-LS2.5-RD, F.Cu at (-15.9, 144.0)
- added D20: A, JLClib:SOD-323_L1.8-W1.3-LS2.5-RD, F.Cu at (-15.9, 146.6)
- added D21: A, JLClib:SOD-323_L1.8-W1.3-LS2.5-RD, F.Cu at (-15.9, 149.2)
- added D22: S, JLClib:SOD-323_L1.8-W1.3-LS2.5-RD, F.Cu at (-15.9, 151.8)
- added D23: A, JLClib:SOD-323_L1.8-W1.3-LS2.5-RD, F.Cu at (-15.9, 154.4)
- added D24: A, JLClib:SOD-323_L1.8-W1.3-LS2.5-RD, F.Cu at (-15.9, 157.0)
- added D25: A, JLClib:SOD-323_L1.8-W1.3-LS2.5-RD, F.Cu at (-15.9, 159.6)
- added D26: A, JLClib:SOD-323_L1.8-W1.3-LS2.5-RD, F.Cu at (-15.9, 162.2)
- added D27: A, JLClib:SOD-323_L1.8-W1.3-LS2.5-RD, F.Cu at (-15.9, 164.9)
- added D28: A, JLClib:SOD-323_L1.8-W1.3-LS2.5-RD, F.Cu at (-11.6, 136.1)
- added D29: A, JLClib:SOD-323_L1.8-W1.3-LS2.5-RD, F.Cu at (-11.6, 138.8)
- added D30: A, JLClib:SOD-323_L1.8-W1.3-LS2.5-RD, F.Cu at (-11.6, 141.4)
- added D31: A, JLClib:SOD-323_L1.8-W1.3-LS2.5-RD, F.Cu at (-11.6, 144.0)
- added D32: A, JLClib:SOD-323_L1.8-W1.3-LS2.5-RD, F.Cu at (-11.6, 146.6)
- added D33: A, JLClib:SOD-323_L1.8-W1.3-LS2.5-RD, F.Cu at (-11.6, 149.2)
- added D34: A, JLClib:SOD-323_L1.8-W1.3-LS2.5-RD, F.Cu at (-11.6, 151.8)
- added D35: A, JLClib:SOD-323_L1.8-W1.3-LS2.5-RD, F.Cu at (-11.6, 154.4)
- added D36: A, JLClib:SOD-323_L1.8-W1.3-LS2.5-RD, F.Cu at (-11.6, 157.0)
- added D37: A, JLClib:SOD-323_L1.8-W1.3-LS2.5-RD, F.Cu at (-11.6, 159.6)
- added D38: A, JLClib:SOD-323_L1.8-W1.3-LS2.5-RD, F.Cu at (-11.6, 162.2)
- added D39: A, JLClib:SOD-323_L1.8-W1.3-LS2.5-RD, F.Cu at (-11.6, 164.9)
- added D4: A, JLClib:SOD-323_L1.8-W1.3-LS2.5-RD, F.Cu at (-20.3, 136.1)
- added D40: A, JLClib:SOD-323_L1.8-W1.3-LS2.5-RD, F.Cu at (-7.25, 136.1)
- added D41: S, JLClib:SOD-323_L1.8-W1.3-LS2.5-RD, F.Cu at (-7.25, 138.8)
- added D42: A, JLClib:SOD-323_L1.8-W1.3-LS2.5-RD, F.Cu at (-7.25, 141.4)
- added D43: A, JLClib:SOD-323_L1.8-W1.3-LS2.5-RD, F.Cu at (-7.25, 144.0)
- added D44: A, JLClib:SOD-323_L1.8-W1.3-LS2.5-RD, F.Cu at (-7.25, 146.6)
- added D45: A, JLClib:SOD-323_L1.8-W1.3-LS2.5-RD, F.Cu at (-7.25, 149.2)
- added D46: A, JLClib:SOD-323_L1.8-W1.3-LS2.5-RD, F.Cu at (-7.25, 151.8)
- added D47: A, JLClib:SOD-323_L1.8-W1.3-LS2.5-RD, F.Cu at (-7.25, 154.4)
- added D48: A, JLClib:SOD-323_L1.8-W1.3-LS2.5-RD, F.Cu at (-7.25, 157.0)
- added D49: A, JLClib:SOD-323_L1.8-W1.3-LS2.5-RD, F.Cu at (-7.25, 159.6)
- added D5: A, JLClib:SOD-323_L1.8-W1.3-LS2.5-RD, F.Cu at (-20.3, 138.8)
- added D50: A, JLClib:SOD-323_L1.8-W1.3-LS2.5-RD, F.Cu at (-7.25, 162.2)
- added D51: A, JLClib:SOD-323_L1.8-W1.3-LS2.5-RD, F.Cu at (-7.25, 164.9)
- added D52: A, JLClib:SOD-323_L1.8-W1.3-LS2.5-RD, F.Cu at (-2.90, 136.1)
- added D53: A, JLClib:SOD-323_L1.8-W1.3-LS2.5-RD, F.Cu at (-2.90, 138.8)
- added D54: A, JLClib:SOD-323_L1.8-W1.3-LS2.5-RD, F.Cu at (-2.90, 141.4)
- added D55: A, JLClib:SOD-323_L1.8-W1.3-LS2.5-RD, F.Cu at (-2.90, 144.0)
- added D56: A, JLClib:SOD-323_L1.8-W1.3-LS2.5-RD, F.Cu at (-2.90, 146.6)
- added D57: S, JLClib:SOD-323_L1.8-W1.3-LS2.5-RD, F.Cu at (-2.90, 149.2)
- added D58: A, JLClib:SOD-323_L1.8-W1.3-LS2.5-RD, F.Cu at (-2.90, 151.8)
- added D59: A, JLClib:SOD-323_L1.8-W1.3-LS2.5-RD, F.Cu at (-2.90, 154.4)
- added D6: A, JLClib:SOD-323_L1.8-W1.3-LS2.5-RD, F.Cu at (-20.3, 141.4)
- added D60: A, JLClib:SOD-323_L1.8-W1.3-LS2.5-RD, F.Cu at (-2.90, 157.0)
- added D61: A, JLClib:SOD-323_L1.8-W1.3-LS2.5-RD, F.Cu at (-2.90, 159.6)
- added D62: A, JLClib:SOD-323_L1.8-W1.3-LS2.5-RD, F.Cu at (-2.90, 162.2)
- added D63: A, JLClib:SOD-323_L1.8-W1.3-LS2.5-RD, F.Cu at (-2.90, 164.9)
- added D64: A, JLClib:SOD-323_L1.8-W1.3-LS2.5-RD, F.Cu at (1.44, 136.1)
- added D65: A, JLClib:SOD-323_L1.8-W1.3-LS2.5-RD, F.Cu at (1.44, 138.8)
- added D66: A, JLClib:SOD-323_L1.8-W1.3-LS2.5-RD, F.Cu at (1.44, 141.4)
- added D67: A, JLClib:SOD-323_L1.8-W1.3-LS2.5-RD, F.Cu at (1.44, 144.0)
- added D68: A, JLClib:SOD-323_L1.8-W1.3-LS2.5-RD, F.Cu at (1.44, 146.6)
- added D69: A, JLClib:SOD-323_L1.8-W1.3-LS2.5-RD, F.Cu at (1.44, 149.2)
- added D7: A, JLClib:SOD-323_L1.8-W1.3-LS2.5-RD, F.Cu at (-20.3, 144.0)
- added D70: A, JLClib:SOD-323_L1.8-W1.3-LS2.5-RD, F.Cu at (1.44, 151.8)
- added D71: A, JLClib:SOD-323_L1.8-W1.3-LS2.5-RD, F.Cu at (1.44, 154.4)
- added D72: A, JLClib:SOD-323_L1.8-W1.3-LS2.5-RD, F.Cu at (1.44, 157.0)
- added D73: A, JLClib:SOD-323_L1.8-W1.3-LS2.5-RD, F.Cu at (1.44, 159.6)
- added D74: S, JLClib:SOD-323_L1.8-W1.3-LS2.5-RD, F.Cu at (1.44, 162.2)
- added D75: A, JLClib:SOD-323_L1.8-W1.3-LS2.5-RD, F.Cu at (1.44, 164.9)
- added D76: A, JLClib:SOD-323_L1.8-W1.3-LS2.5-RD, F.Cu at (5.78, 136.1)
- added D77: A, JLClib:SOD-323_L1.8-W1.3-LS2.5-RD, F.Cu at (5.78, 138.8)
- added D78: A, JLClib:SOD-323_L1.8-W1.3-LS2.5-RD, F.Cu at (5.78, 141.4)
- added D79: A, JLClib:SOD-323_L1.8-W1.3-LS2.5-RD, F.Cu at (5.78, 144.0)
- added D8: A, JLClib:SOD-323_L1.8-W1.3-LS2.5-RD, F.Cu at (-20.3, 146.6)
- added D80: A, JLClib:SOD-323_L1.8-W1.3-LS2.5-RD, F.Cu at (5.78, 146.6)
- added D81: A, JLClib:SOD-323_L1.8-W1.3-LS2.5-RD, F.Cu at (5.78, 149.2)
- added D82: A, JLClib:SOD-323_L1.8-W1.3-LS2.5-RD, F.Cu at (5.78, 151.8)
- added D83: A, JLClib:SOD-323_L1.8-W1.3-LS2.5-RD, F.Cu at (5.78, 154.4)
- added D9: A, JLClib:SOD-323_L1.8-W1.3-LS2.5-RD, F.Cu at (-20.3, 149.2)
- added K10: 100nF, JLClib:C0402, F.Cu at (27.9, 177.8)
- added K11: 100nF, JLClib:C0402, F.Cu at (27.9, 180.0)
- added K12: 100nF, JLClib:C0402, F.Cu at (27.9, 182.1)
- added K13: 100nF, JLClib:C0402, F.Cu at (27.9, 184.3)
- added K14: 100nF, JLClib:C0402, F.Cu at (27.9, 186.4)
- added K15: 100nF, JLClib:C0402, F.Cu at (27.9, 188.6)
- added K16: 100nF, JLClib:C0402, F.Cu at (27.9, 190.7)
- added K17: 100nF, JLClib:C0402, F.Cu at (27.9, 192.9)
- added K18: 100nF, JLClib:C0402, F.Cu at (27.9, 195.0)
- added K19: 100nF, JLClib:C0402, F.Cu at (31.4, 169.2)
- added K20: 100nF, JLClib:C0402, F.Cu at (31.4, 171.4)
- added K21: 100nF, JLClib:C0402, F.Cu at (31.4, 173.5)
- added K22: 100nF, JLClib:C0402, F.Cu at (31.4, 175.7)
- added K23: 100nF, JLClib:C0402, F.Cu at (31.4, 177.8)
- added K24: 100nF, JLClib:C0402, F.Cu at (31.4, 180.0)
- added K25: 100nF, JLClib:C0402, F.Cu at (31.4, 182.1)
- added K26: 100nF, JLClib:C0402, F.Cu at (31.4, 184.3)
- added K27: 100nF, JLClib:C0402, F.Cu at (31.4, 186.4)
- added K28: 100nF, JLClib:C0402, F.Cu at (31.4, 188.6)
- added K29: 100nF, JLClib:C0402, F.Cu at (31.4, 190.7)
- added K30: 100nF, JLClib:C0402, F.Cu at (31.4, 192.9)
- added K31: 100nF, JLClib:C0402, F.Cu at (31.4, 195.0)
- added K32: 100nF, JLClib:C0402, F.Cu at (34.9, 169.2)
- added K33: 100nF, JLClib:C0402, F.Cu at (34.9, 171.4)
- added K34: 100nF, JLClib:C0402, F.Cu at (34.9, 173.5)
- added K35: 100nF, JLClib:C0402, F.Cu at (34.9, 175.7)
- added K36: 100nF, JLClib:C0402, F.Cu at (34.9, 177.8)
- added K37: 100nF, JLClib:C0402, F.Cu at (34.9, 180.0)
- added K38: 100nF, JLClib:C0402, F.Cu at (34.9, 182.1)
- added K39: 100nF, JLClib:C0402, F.Cu at (34.9, 184.3)
- added K40: 100nF, JLClib:C0402, F.Cu at (34.9, 186.4)
- added K41: 100nF, JLClib:C0402, F.Cu at (34.9, 188.6)
- added K42: 100nF, JLClib:C0402, F.Cu at (34.9, 190.7)
- added K43: 100nF, JLClib:C0402, F.Cu at (34.9, 192.9)
- added K44: 100nF, JLClib:C0402, F.Cu at (34.9, 195.0)
- added K45: 100nF, JLClib:C0402, F.Cu at (38.4, 169.2)
- added K46: 100nF, JLClib:C0402, F.Cu at (38.4, 171.4)
- added K47: 100nF, JLClib:C0402, F.Cu at (38.4, 173.5)
- added K48: 100nF, JLClib:C0402, F.Cu at (38.4, 175.7)
- added K49: 100nF, JLClib:C0402, F.Cu at (38.4, 177.8)
- added K50: 100nF, JLClib:C0402, F.Cu at (38.4, 180.0)
- added K51: 100nF, JLClib:C0402, F.Cu at (38.4, 182.1)
- added K52: 100nF, JLClib:C0402, F.Cu at (38.4, 184.3)
- added K53: 100nF, JLClib:C0402, F.Cu at (38.4, 186.4)
- added K54: 100nF, JLClib:C0402, F.Cu at (38.4, 188.6)
- added K55: 100nF, JLClib:C0402, F.Cu at (38.4, 190.7)
- added K59: 100nF, JLClib:C0402, F.Cu at (38.4, 192.9)
- added K6: 100nF, JLClib:C0402, F.Cu at (27.9, 169.2)
- added K60: 100nF, JLClib:C0402, F.Cu at (38.4, 195.0)
- added K61: 100nF, JLClib:C0402, F.Cu at (41.9, 169.2)
- added K62: 100nF, JLClib:C0402, F.Cu at (41.9, 171.4)
- added K63: 100nF, JLClib:C0402, F.Cu at (41.9, 173.5)
- added K64: 100nF, JLClib:C0402, F.Cu at (41.9, 175.7)
- added K65: 100nF, JLClib:C0402, F.Cu at (41.9, 177.8)
- added K66: 100nF, JLClib:C0402, F.Cu at (41.9, 180.0)
- added K67: 100nF, JLClib:C0402, F.Cu at (41.9, 182.1)
- added K68: 100nF, JLClib:C0402, F.Cu at (41.9, 184.3)
- added K69: 100nF, JLClib:C0402, F.Cu at (41.9, 186.4)
- added K7: 100nF, JLClib:C0402, F.Cu at (27.9, 171.4)
- added K70: 100nF, JLClib:C0402, F.Cu at (41.9, 188.6)
- added K71: 100nF, JLClib:C0402, F.Cu at (41.9, 190.7)
- added K72: 100nF, JLClib:C0402, F.Cu at (41.9, 192.9)
- added K73: 100nF, JLClib:C0402, F.Cu at (41.9, 195.0)
- added K74: 100nF, JLClib:C0402, F.Cu at (45.4, 169.2)
- added K75: 100nF, JLClib:C0402, F.Cu at (45.4, 171.4)
- added K78: 100nF, JLClib:C0402, F.Cu at (45.4, 173.5)
- added K79: 100nF, JLClib:C0402, F.Cu at (45.4, 175.7)
- added K8: 100nF, JLClib:C0402, F.Cu at (27.9, 173.5)
- added K80: 100nF, JLClib:C0402, F.Cu at (45.4, 177.8)
- added K81: 100nF, JLClib:C0402, F.Cu at (45.4, 180.0)
- added K82: 100nF, JLClib:C0402, F.Cu at (45.4, 182.1)
- added K83: 100nF, JLClib:C0402, F.Cu at (45.4, 184.3)
- added K84: 100nF, JLClib:C0402, F.Cu at (45.4, 186.4)
- added K85: 100nF, JLClib:C0402, F.Cu at (45.4, 188.6)
- added K86: 100nF, JLClib:C0402, F.Cu at (45.4, 190.7)
- added K87: 100nF, JLClib:C0402, F.Cu at (45.4, 192.9)
- added K88: 100nF, JLClib:C0402, F.Cu at (45.4, 195.0)
- added K9: 100nF, JLClib:C0402, F.Cu at (27.9, 175.7)
- added SW10: ~, JLClib:SW_Cherry_MX_1.00u_Plate, F.Cu at (-14.9, 112.2)
- added SW11: ~, JLClib:SW_Cherry_MX_1.00u_Plate, F.Cu at (-14.9, 127.3)
- added SW12: ~, JLClib:SW_Cherry_MX_1.00u_Plate, F.Cu at (0.20, 21.7)
- added SW13: ~, JLClib:SW_Cherry_MX_1.00u_Plate, F.Cu at (0.20, 36.8)
- added SW14: ~, JLClib:SW_Cherry_MX_1.00u_Plate, F.Cu at (0.20, 51.8)
- added SW15: ~, JLClib:SW_Cherry_MX_1.00u_Plate, F.Cu at (0.20, 66.9)
- added SW16: ~, JLClib:SW_Cherry_MX_1.00u_Plate, F.Cu at (0.20, 82.0)
- added SW17: ~, JLClib:SW_Cherry_MX_1.00u_Plate, F.Cu at (0.20, 97.1)
- added SW18: ~, JLClib:SW_Cherry_MX_1.00u_Plate, F.Cu at (0.20, 112.2)
- added SW19: ~, JLClib:SW_Cherry_MX_1.00u_Plate, F.Cu at (0.20, 127.3)
- added SW20: ~, JLClib:SW_Cherry_MX_1.00u_Plate, F.Cu at (15.3, 21.7)
- added SW21: ~, JLClib:SW_Cherry_MX_1.00u_Plate, F.Cu at (15.3, 36.8)
- added SW22: ~, JLClib:SW_Cherry_MX_1.00u_Plate, F.Cu at (15.3, 51.8)
- added SW23: ~, JLClib:SW_Cherry_MX_1.00u_Plate, F.Cu at (15.3, 66.9)
- added SW24: ~, JLClib:SW_Cherry_MX_1.00u_Plate, F.Cu at (15.3, 82.0)
- added SW25: ~, JLClib:SW_Cherry_MX_1.00u_Plate, F.Cu at (15.3, 97.1)
- added SW26: ~, JLClib:SW_Cherry_MX_1.00u_Plate, F.Cu at (15.3, 112.2)
- added SW27: ~, JLClib:SW_Cherry_MX_1.00u_Plate, F.Cu at (15.3, 127.3)
- added SW28: ~, JLClib:SW_Cherry_MX_1.00u_Plate, F.Cu at (30.4, 21.7)
- added SW29: ~, JLClib:SW_Cherry_MX_1.00u_Plate, F.Cu at (30.4, 36.8)
- added SW30: ~, JLClib:SW_Cherry_MX_1.00u_Plate, F.Cu at (30.4, 51.8)
- added SW31: ~, JLClib:SW_Cherry_MX_1.00u_Plate, F.Cu at (30.4, 66.9)
- added SW32: ~, JLClib:SW_Cherry_MX_1.00u_Plate, F.Cu at (30.4, 82.0)
- added SW33: ~, JLClib:SW_Cherry_MX_1.00u_Plate, F.Cu at (30.4, 97.1)
- added SW34: ~, JLClib:SW_Cherry_MX_1.00u_Plate, F.Cu at (30.4, 112.2)
- added SW35: ~, JLClib:SW_Cherry_MX_1.00u_Plate, F.Cu at (30.4, 127.3)
- added SW36: ~, JLClib:SW_Cherry_MX_1.00u_Plate, F.Cu at (45.5, 21.7)
- added SW37: ~, JLClib:SW_Cherry_MX_1.00u_Plate, F.Cu at (45.5, 36.8)
- added SW38: ~, JLClib:SW_Cherry_MX_1.00u_Plate, F.Cu at (45.5, 51.8)
- added SW39: ~, JLClib:SW_Cherry_MX_1.00u_Plate, F.Cu at (45.5, 66.9)
- added SW4: ~, JLClib:SW_Cherry_MX_1.00u_Plate, F.Cu at (-14.9, 21.7)
- added SW40: ~, JLClib:SW_Cherry_MX_1.00u_Plate, F.Cu at (45.5, 82.0)
- added SW41: ~, JLClib:SW_Cherry_MX_1.00u_Plate, F.Cu at (45.5, 97.1)
- added SW42: ~, JLClib:SW_Cherry_MX_1.00u_Plate, F.Cu at (45.5, 112.2)
- added SW43: ~, JLClib:SW_Cherry_MX_1.00u_Plate, F.Cu at (45.5, 127.3)
- added SW44: ~, JLClib:SW_Cherry_MX_1.00u_Plate, F.Cu at (60.6, 21.7)
- added SW45: ~, JLClib:SW_Cherry_MX_1.00u_Plate, F.Cu at (60.6, 36.8)
- added SW46: ~, JLClib:SW_Cherry_MX_1.00u_Plate, F.Cu at (60.6, 51.8)
- added SW47: ~, JLClib:SW_Cherry_MX_1.00u_Plate, F.Cu at (60.6, 66.9)
- added SW48: ~, JLClib:SW_Cherry_MX_1.00u_Plate, F.Cu at (60.6, 82.0)
- added SW49: ~, JLClib:SW_Cherry_MX_1.00u_Plate, F.Cu at (60.6, 97.1)
- added SW5: ~, JLClib:SW_Cherry_MX_1.00u_Plate, F.Cu at (-14.9, 36.8)
- added SW50: ~, JLClib:SW_Cherry_MX_1.00u_Plate, F.Cu at (60.6, 112.2)
- added SW51: ~, JLClib:SW_Cherry_MX_1.00u_Plate, F.Cu at (60.6, 127.3)
- added SW52: ~, JLClib:SW_Cherry_MX_1.00u_Plate, F.Cu at (75.7, 21.7)
- added SW53: ~, JLClib:SW_Cherry_MX_1.00u_Plate, F.Cu at (75.7, 36.8)
- added SW54: ~, JLClib:SW_Cherry_MX_1.00u_Plate, F.Cu at (75.7, 51.8)
- added SW55: ~, JLClib:SW_Cherry_MX_1.00u_Plate, F.Cu at (75.7, 66.9)
- added SW56: ~, JLClib:SW_Cherry_MX_1.00u_Plate, F.Cu at (75.7, 82.0)
- added SW57: ~, JLClib:SW_Cherry_MX_1.00u_Plate, F.Cu at (75.7, 97.1)
- added SW58: ~, JLClib:SW_Cherry_MX_1.00u_Plate, F.Cu at (75.7, 112.2)
- added SW59: ~, JLClib:SW_Cherry_MX_1.00u_Plate, F.Cu at (75.7, 127.3)
- added SW6: ~, JLClib:SW_Cherry_MX_1.00u_Plate, F.Cu at (-14.9, 51.8)
- added SW60: ~, JLClib:SW_Cherry_MX_1.00u_Plate, F.Cu at (90.7, 21.7)
- added SW61: ~, JLClib:SW_Cherry_MX_1.00u_Plate, F.Cu at (90.7, 36.8)
- added SW62: ~, JLClib:SW_Cherry_MX_1.00u_Plate, F.Cu at (90.7, 51.8)
- added SW63: ~, JLClib:SW_Cherry_MX_1.00u_Plate, F.Cu at (90.7, 66.9)
- added SW64: ~, JLClib:SW_Cherry_MX_1.00u_Plate, F.Cu at (90.7, 82.0)
- added SW65: ~, JLClib:SW_Cherry_MX_1.00u_Plate, F.Cu at (90.7, 97.1)
- added SW66: ~, JLClib:SW_Cherry_MX_1.00u_Plate, F.Cu at (90.7, 112.2)
- added SW67: ~, JLClib:SW_Cherry_MX_1.00u_Plate, F.Cu at (90.7, 127.3)
- added SW68: ~, JLClib:SW_Cherry_MX_1.00u_Plate, F.Cu at (105.8, 21.7)
- added SW69: ~, JLClib:SW_Cherry_MX_1.00u_Plate, F.Cu at (105.8, 36.8)
- added SW7: ~, JLClib:SW_Cherry_MX_1.00u_Plate, F.Cu at (-14.9, 66.9)
- added SW70: ~, JLClib:SW_Cherry_MX_1.00u_Plate, F.Cu at (105.8, 51.8)
- added SW71: ~, JLClib:SW_Cherry_MX_1.00u_Plate, F.Cu at (105.8, 66.9)
- added SW72: ~, JLClib:SW_Cherry_MX_1.00u_Plate, F.Cu at (105.8, 82.0)
- added SW73: ~, JLClib:SW_Cherry_MX_1.00u_Plate, F.Cu at (105.8, 97.1)
- added SW74: ~, JLClib:SW_Cherry_MX_1.00u_Plate, F.Cu at (105.8, 112.2)
- added SW75: ~, JLClib:SW_Cherry_MX_1.00u_Plate, F.Cu at (105.8, 127.3)
- added SW76: ~, JLClib:SW_Cherry_MX_1.00u_Plate, F.Cu at (120.9, 21.7)
- added SW77: ~, JLClib:SW_Cherry_MX_1.00u_Plate, F.Cu at (120.9, 36.8)
- added SW78: ~, JLClib:SW_Cherry_MX_1.00u_Plate, F.Cu at (120.9, 51.8)
- added SW79: ~, JLClib:SW_Cherry_MX_1.00u_Plate, F.Cu at (120.9, 66.9)
- added SW8: ~, JLClib:SW_Cherry_MX_1.00u_Plate, F.Cu at (-14.9, 82.0)
- added SW80: ~, JLClib:SW_Cherry_MX_1.00u_Plate, F.Cu at (120.9, 82.0)
- added SW81: ~, JLClib:SW_Cherry_MX_1.00u_Plate, F.Cu at (120.9, 97.1)
- added SW82: ~, JLClib:SW_Cherry_MX_1.00u_Plate, F.Cu at (120.9, 112.2)
- added SW83: ~, JLClib:SW_Cherry_MX_1.00u_Plate, F.Cu at (120.9, 127.3)
- added SW9: ~, JLClib:SW_Cherry_MX_1.00u_Plate, F.Cu at (-14.9, 97.1)
- added U10: ~, JLClib:LED-SMD_L3.2-W2.8-TR, F.Cu at (-18.4, 195.9)
- added U11: ~, JLClib:LED-SMD_L3.2-W2.8-TR, F.Cu at (-18.4, 200.1)
- added U12: ~, JLClib:LED-SMD_L3.2-W2.8-TR, F.Cu at (-18.4, 204.4)
- added U13: ~, JLClib:LED-SMD_L3.2-W2.8-TR, F.Cu at (-18.4, 208.6)
- added U14: ~, JLClib:LED-SMD_L3.2-W2.8-TR, F.Cu at (-18.4, 212.9)
- added U15: ~, JLClib:LED-SMD_L3.2-W2.8-TR, F.Cu at (-18.4, 217.2)
- added U16: ~, JLClib:LED-SMD_L3.2-W2.8-TR, F.Cu at (-18.4, 221.4)
- added U17: ~, JLClib:LED-SMD_L3.2-W2.8-TR, F.Cu at (-18.4, 225.7)
- added U18: ~, JLClib:LED-SMD_L3.2-W2.8-TR, F.Cu at (-10.3, 170.3)
- added U19: ~, JLClib:LED-SMD_L3.2-W2.8-TR, F.Cu at (-10.3, 174.6)
- added U20: ~, JLClib:LED-SMD_L3.2-W2.8-TR, F.Cu at (-10.3, 178.8)
- added U21: ~, JLClib:LED-SMD_L3.2-W2.8-TR, F.Cu at (-10.3, 183.1)
- added U22: ~, JLClib:LED-SMD_L3.2-W2.8-TR, F.Cu at (-10.3, 187.3)
- added U23: ~, JLClib:LED-SMD_L3.2-W2.8-TR, F.Cu at (-10.3, 191.6)
- added U24: ~, JLClib:LED-SMD_L3.2-W2.8-TR, F.Cu at (-10.3, 195.9)
- added U25: ~, JLClib:LED-SMD_L3.2-W2.8-TR, F.Cu at (-10.3, 200.1)
- added U26: ~, JLClib:LED-SMD_L3.2-W2.8-TR, F.Cu at (-10.3, 204.4)
- added U27: ~, JLClib:LED-SMD_L3.2-W2.8-TR, F.Cu at (-10.3, 208.6)
- added U28: ~, JLClib:LED-SMD_L3.2-W2.8-TR, F.Cu at (-10.3, 212.9)
- added U29: ~, JLClib:LED-SMD_L3.2-W2.8-TR, F.Cu at (-10.3, 217.2)
- added U30: ~, JLClib:LED-SMD_L3.2-W2.8-TR, F.Cu at (-10.3, 221.4)
- added U31: ~, JLClib:LED-SMD_L3.2-W2.8-TR, F.Cu at (-10.3, 225.7)
- added U32: ~, JLClib:LED-SMD_L3.2-W2.8-TR, F.Cu at (-2.19, 170.3)
- added U33: ~, JLClib:LED-SMD_L3.2-W2.8-TR, F.Cu at (-2.19, 174.6)
- added U34: ~, JLClib:LED-SMD_L3.2-W2.8-TR, F.Cu at (-2.19, 178.8)
- added U35: ~, JLClib:LED-SMD_L3.2-W2.8-TR, F.Cu at (-2.19, 183.1)
- added U36: ~, JLClib:LED-SMD_L3.2-W2.8-TR, F.Cu at (-2.19, 187.3)
- added U37: ~, JLClib:LED-SMD_L3.2-W2.8-TR, F.Cu at (-2.19, 191.6)
- added U38: ~, JLClib:LED-SMD_L3.2-W2.8-TR, F.Cu at (-2.19, 195.9)
- added U39: ~, JLClib:LED-SMD_L3.2-W2.8-TR, F.Cu at (-2.19, 200.1)
- added U4: ~, JLClib:LED-SMD_L3.2-W2.8-TR, F.Cu at (-18.4, 170.3)
- added U40: ~, JLClib:LED-SMD_L3.2-W2.8-TR, F.Cu at (-2.19, 204.4)
- added U41: ~, JLClib:LED-SMD_L3.2-W2.8-TR, F.Cu at (-2.19, 208.6)
- added U42: ~, JLClib:LED-SMD_L3.2-W2.8-TR, F.Cu at (-2.19, 212.9)
- added U43: ~, JLClib:LED-SMD_L3.2-W2.8-TR, F.Cu at (-2.19, 217.2)
- added U44: ~, JLClib:LED-SMD_L3.2-W2.8-TR, F.Cu at (-2.19, 221.4)
- added U45: ~, JLClib:LED-SMD_L3.2-W2.8-TR, F.Cu at (-2.19, 225.7)
- added U46: ~, JLClib:LED-SMD_L3.2-W2.8-TR, F.Cu at (5.92, 170.3)
- added U47: ~, JLClib:LED-SMD_L3.2-W2.8-TR, F.Cu at (5.92, 174.6)
- added U48: ~, JLClib:LED-SMD_L3.2-W2.8-TR, F.Cu at (5.92, 178.8)
- added U49: ~, JLClib:LED-SMD_L3.2-W2.8-TR, F.Cu at (5.92, 183.1)
- added U5: ~, JLClib:LED-SMD_L3.2-W2.8-TR, F.Cu at (-18.4, 174.6)
- added U50: ~, JLClib:LED-SMD_L3.2-W2.8-TR, F.Cu at (5.92, 187.3)
- added U51: ~, JLClib:LED-SMD_L3.2-W2.8-TR, F.Cu at (5.92, 191.6)
- added U52: ~, JLClib:LED-SMD_L3.2-W2.8-TR, F.Cu at (5.92, 195.9)
- added U53: ~, JLClib:LED-SMD_L3.2-W2.8-TR, F.Cu at (5.92, 200.1)
- added U54: ~, JLClib:LED-SMD_L3.2-W2.8-TR, F.Cu at (5.92, 204.4)
- added U55: ~, JLClib:LED-SMD_L3.2-W2.8-TR, F.Cu at (5.92, 208.6)
- added U56: ~, JLClib:LED-SMD_L3.2-W2.8-TR, F.Cu at (5.92, 212.9)
- added U57: ~, JLClib:LED-SMD_L3.2-W2.8-TR, F.Cu at (5.92, 217.2)
- added U58: ~, JLClib:LED-SMD_L3.2-W2.8-TR, F.Cu at (5.92, 221.4)
- added U59: ~, JLClib:LED-SMD_L3.2-W2.8-TR, F.Cu at (5.92, 225.7)
- added U6: ~, JLClib:LED-SMD_L3.2-W2.8-TR, F.Cu at (-18.4, 178.8)
- added U60: ~, JLClib:LED-SMD_L3.2-W2.8-TR, F.Cu at (14.0, 170.3)
- added U61: ~, JLClib:LED-SMD_L3.2-W2.8-TR, F.Cu at (14.0, 174.6)
- added U62: ~, JLClib:LED-SMD_L3.2-W2.8-TR, F.Cu at (14.0, 178.8)
- added U63: ~, JLClib:LED-SMD_L3.2-W2.8-TR, F.Cu at (14.0, 183.1)
- added U64: ~, JLClib:LED-SMD_L3.2-W2.8-TR, F.Cu at (14.0, 187.3)
- added U65: ~, JLClib:LED-SMD_L3.2-W2.8-TR, F.Cu at (14.0, 191.6)
- added U66: ~, JLClib:LED-SMD_L3.2-W2.8-TR, F.Cu at (14.0, 195.9)
- added U67: ~, JLClib:LED-SMD_L3.2-W2.8-TR, F.Cu at (14.0, 200.1)
- added U68: ~, JLClib:LED-SMD_L3.2-W2.8-TR, F.Cu at (14.0, 204.4)
- added U69: ~, JLClib:LED-SMD_L3.2-W2.8-TR, F.Cu at (14.0, 208.6)
- added U7: ~, JLClib:LED-SMD_L3.2-W2.8-TR, F.Cu at (-18.4, 183.1)
- added U70: ~, JLClib:LED-SMD_L3.2-W2.8-TR, F.Cu at (14.0, 212.9)
- added U71: ~, JLClib:LED-SMD_L3.2-W2.8-TR, F.Cu at (14.0, 217.2)
- added U72: ~, JLClib:LED-SMD_L3.2-W2.8-TR, F.Cu at (14.0, 221.4)
- added U73: ~, JLClib:LED-SMD_L3.2-W2.8-TR, F.Cu at (14.0, 225.7)
- added U74: ~, JLClib:LED-SMD_L3.2-W2.8-TR, F.Cu at (22.1, 170.3)
- added U75: ~, JLClib:LED-SMD_L3.2-W2.8-TR, F.Cu at (22.1, 174.6)
- added U76: ~, JLClib:LED-SMD_L3.2-W2.8-TR, F.Cu at (22.1, 178.8)
- added U77: ~, JLClib:LED-SMD_L3.2-W2.8-TR, F.Cu at (22.1, 183.1)
- added U78: ~, JLClib:LED-SMD_L3.2-W2.8-TR, F.Cu at (22.1, 187.3)
- added U79: ~, JLClib:LED-SMD_L3.2-W2.8-TR, F.Cu at (22.1, 191.6)
- added U8: ~, JLClib:LED-SMD_L3.2-W2.8-TR, F.Cu at (-18.4, 187.3)
- added U80: ~, JLClib:LED-SMD_L3.2-W2.8-TR, F.Cu at (22.1, 195.9)
- added U81: ~, JLClib:LED-SMD_L3.2-W2.8-TR, F.Cu at (22.1, 200.1)
- added U82: ~, JLClib:LED-SMD_L3.2-W2.8-TR, F.Cu at (22.1, 204.4)
- added U83: ~, JLClib:LED-SMD_L3.2-W2.8-TR, F.Cu at (22.1, 208.6)
- added U9: ~, JLClib:LED-SMD_L3.2-W2.8-TR, F.Cu at (-18.4, 191.6)
- SW1: value ~ -> Boot Switch
- SW2: value A -> ~
- SW3: value S -> ~
- U2: renamed from U3; value A -> ~
- U3: renamed from U5; value S -> ~
- renumbered C11 to K2, C12 to K3, C13 to K4, C14 to K5, U1 to X1, U2 to X2
Connections:
- R1 pad 1: Net-(SW1-D) -> GND
- R1 pad 2: /STM32/Boot -> Net-(SW1-C)
- SW1 pad 3: GND -> Net-(SW1-C)
- SW1 pad 4: Net-(SW1-D) -> /STM32/Boot
- U2 pad 1: +5V -> Net-(U10-VDD)
- U3 pad 1: +5V -> Net-(U10-VDD)
- U3 pad 2: Net-(U5-DOUT) -> Net-(U3-DOUT)
- X1 pad 10: unconnected-(U1-PA0-Pad10) -> /Keyboard Matrix/Row0
- X1 pad 11: unconnected-(U1-PA1-Pad11) -> /Keyboard Matrix/Col13
- X1 pad 12: unconnected-(U1-PA2-Pad12) -> /Keyboard Matrix/Col14
- X1 pad 13: unconnected-(U1-PA3-Pad13) -> /Keyboard Matrix/Col15
- X1 pad 14: unconnected-(U1-PA4-Pad14) -> /Keyboard Matrix/Col16
- X1 pad 15: unconnected-(U1-PA5-Pad15) -> /Keyboard Matrix/Col17
- X1 pad 16: unconnected-(U1-PA6-Pad16) -> /Keyboard Matrix/Col18
- X1 pad 17: unconnected-(U1-PA7-Pad17) -> /RGB LEDs/LED_Control
- X1 pad 25: Net-(U1-PB12) -> /Keyboard Matrix/Col12
- X1 pad 26: Net-(U1-PB13) -> /Keyboard Matrix/Col11
- X1 pad 27: Net-(U1-PB14) -> /Keyboard Matrix/Col10
- X1 pad 28: Net-(U1-PB15) -> /Keyboard Matrix/Col9
- X1 pad 29: unconnected-(U1-PA8-Pad29) -> /Keyboard Matrix/Col8
- X1 pad 30: unconnected-(U1-PA9-Pad30) -> /Keyboard Matrix/Col7
- X1 pad 31: unconnected-(U1-PA10-Pad31) -> /Keyboard Matrix/Col6
- X1 pad 34: unconnected-(U1-PA13-Pad34) -> /Keyboard Matrix/Col5
- X1 pad 37: /Keyboard Matrix/Col0 -> /Keyboard Matrix/Col4
- X1 pad 38: /Keyboard Matrix/Col1 -> /Keyboard Matrix/Col3
- X1 pad 39: /Keyboard Matrix/Row0 -> /Keyboard Matrix/Col2
- X1 pad 40: /Keyboard Matrix/Row1 -> /Keyboard Matrix/Col1
- X1 pad 41: /RGB LEDs/LED_Control -> /Keyboard Matrix/Col0
- X1 pad 42: unconnected-(U1-PB6-Pad42) -> /Keyboard Matrix/Row4
- X1 pad 43: unconnected-(U1-PB7-Pad43) -> /Keyboard Matrix/Row3
- X1 pad 45: unconnected-(U1-PB8-Pad45) -> /Keyboard Matrix/Row2
- X1 pad 46: unconnected-(U1-PB9-Pad46) -> /Keyboard Matrix/Row1
Routing:
- net Net-(SW1-D): track 9.47 -> 0.00 mm, vias 1 -> 0
- net (no net): track 0.00 -> 9.47 mm
- net /STM32/Boot: vias 0 -> 1

Commit message: Board scripting
Parts:
- removed the SW4 at (188.0, 76.5)
- added D68: A, JLClib:SOD-323_L1.8-W1.3-LS2.5-RD, F.Cu at (235.7, 57.1)
- added K73: 100nF, JLClib:C0402, F.Cu at (362.0, 66.7)
- added SW68: Shift, Button_Switch_Keyboard:SW_Cherry_MX_1.25u_Plate, F.Cu at (235.7, 57.1)
- added U73: ~, JLClib:LED-SMD_L3.2-W2.8-TR, F.Cu at (361.9, 66.7)
- SW10: value ~ -> * 8; footprint JLClib:SW_Cherry_MX_1.00u_Plate -> Button_Switch_Keyboard:SW_Cherry_MX_1.00u_Plate
- SW11: value ~ -> ( 9; footprint JLClib:SW_Cherry_MX_1.00u_Plate -> Button_Switch_Keyboard:SW_Cherry_MX_1.00u_Plate
- SW12: value ~ -> ) 0; footprint JLClib:SW_Cherry_MX_1.00u_Plate -> Button_Switch_Keyboard:SW_Cherry_MX_1.00u_Plate
- SW13: value ~ -> _ -; footprint JLClib:SW_Cherry_MX_1.00u_Plate -> Button_Switch_Keyboard:SW_Cherry_MX_1.00u_Plate
- SW14: value ~ -> + =; footprint JLClib:SW_Cherry_MX_1.00u_Plate -> Button_Switch_Keyboard:SW_Cherry_MX_1.00u_Plate
- SW15: value ~ -> Backspace; footprint JLClib:SW_Cherry_MX_1.00u_Plate -> Button_Switch_Keyboard:SW_Cherry_MX_2.00u_Plate
- SW16: value ~ -> Insert; footprint JLClib:SW_Cherry_MX_1.00u_Plate -> Button_Switch_Keyboard:SW_Cherry_MX_1.00u_Plate
- SW17: value ~ -> %; footprint JLClib:SW_Cherry_MX_1.00u_Plate -> Button_Switch_Keyboard:SW_Cherry_MX_1.00u_Plate
- SW18: value ~ -> /; footprint JLClib:SW_Cherry_MX_1.00u_Plate -> Button_Switch_Keyboard:SW_Cherry_MX_1.00u_Plate
- SW19: value ~ -> *; footprint JLClib:SW_Cherry_MX_1.00u_Plate -> Button_Switch_Keyboard:SW_Cherry_MX_1.00u_Plate
- SW2: value ~ -> Esc; footprint JLClib:SW_Cherry_MX_1.00u_Plate -> Button_Switch_Keyboard:SW_Cherry_MX_1.00u_Plate
- SW20: value ~ -> -; footprint JLClib:SW_Cherry_MX_1.00u_Plate -> Button_Switch_Keyboard:SW_Cherry_MX_1.00u_Plate
- SW21: value ~ -> Tab; footprint JLClib:SW_Cherry_MX_1.00u_Plate -> Button_Switch_Keyboard:SW_Cherry_MX_1.50u_Plate
- SW22: value ~ -> Q; footprint JLClib:SW_Cherry_MX_1.00u_Plate -> Button_Switch_Keyboard:SW_Cherry_MX_1.00u_Plate
- SW23: value ~ -> W; footprint JLClib:SW_Cherry_MX_1.00u_Plate -> Button_Switch_Keyboard:SW_Cherry_MX_1.00u_Plate
- SW24: value ~ -> E; footprint JLClib:SW_Cherry_MX_1.00u_Plate -> Button_Switch_Keyboard:SW_Cherry_MX_1.00u_Plate
- SW25: value ~ -> R; footprint JLClib:SW_Cherry_MX_1.00u_Plate -> Button_Switch_Keyboard:SW_Cherry_MX_1.00u_Plate
- SW26: value ~ -> T; footprint JLClib:SW_Cherry_MX_1.00u_Plate -> Button_Switch_Keyboard:SW_Cherry_MX_1.00u_Plate
- SW27: value ~ -> Y; footprint JLClib:SW_Cherry_MX_1.00u_Plate -> Button_Switch_Keyboard:SW_Cherry_MX_1.00u_Plate
- SW28: value ~ -> U; footprint JLClib:SW_Cherry_MX_1.00u_Plate -> Button_Switch_Keyboard:SW_Cherry_MX_1.00u_Plate
- SW29: value ~ -> I; footprint JLClib:SW_Cherry_MX_1.00u_Plate -> Button_Switch_Keyboard:SW_Cherry_MX_1.00u_Plate
- SW3: value ~ -> ! 1; footprint JLClib:SW_Cherry_MX_1.00u_Plate -> Button_Switch_Keyboard:SW_Cherry_MX_1.00u_Plate
- SW30: value ~ -> O; footprint JLClib:SW_Cherry_MX_1.00u_Plate -> Button_Switch_Keyboard:SW_Cherry_MX_1.00u_Plate
- SW31: value ~ -> P; footprint JLClib:SW_Cherry_MX_1.00u_Plate -> Button_Switch_Keyboard:SW_Cherry_MX_1.00u_Plate
- SW32: value ~ -> { [; footprint JLClib:SW_Cherry_MX_1.00u_Plate -> Button_Switch_Keyboard:SW_Cherry_MX_1.00u_Plate
- SW33: value ~ -> } ]; footprint JLClib:SW_Cherry_MX_1.00u_Plate -> Button_Switch_Keyboard:SW_Cherry_MX_1.00u_Plate
- SW34: value ~ -> Enter; footprint JLClib:SW_Cherry_MX_1.00u_Plate -> Button_Switch_Keyboard:SW_Cherry_MX_ISOEnter_Plate
- SW35: value ~ -> Delete; footprint JLClib:SW_Cherry_MX_1.00u_Plate -> Button_Switch_Keyboard:SW_Cherry_MX_1.00u_Plate
- SW36: value ~ -> 7 Home; footprint JLClib:SW_Cherry_MX_1.00u_Plate -> Button_Switch_Keyboard:SW_Cherry_MX_1.00u_Plate
- SW37: value ~ -> 8 ↑; footprint JLClib:SW_Cherry_MX_1.00u_Plate -> Button_Switch_Keyboard:SW_Cherry_MX_1.00u_Plate
- SW38: value ~ -> 9 PgUp; footprint JLClib:SW_Cherry_MX_1.00u_Plate -> Button_Switch_Keyboard:SW_Cherry_MX_1.00u_Plate
- SW39: value ~ -> +; footprint JLClib:SW_Cherry_MX_1.00u_Plate -> Button_Switch_Keyboard:SW_Cherry_MX_2.00u_Vertical_Plate
- SW4: value ~ -> " 2; footprint JLClib:SW_Cherry_MX_1.00u_Plate -> Button_Switch_Keyboard:SW_Cherry_MX_1.00u_Plate
- SW40: value ~ -> Caps Lock; footprint JLClib:SW_Cherry_MX_1.00u_Plate -> Button_Switch_Keyboard:SW_Cherry_MX_1.75u_Plate
- SW41: value ~ -> A; footprint JLClib:SW_Cherry_MX_1.00u_Plate -> Button_Switch_Keyboard:SW_Cherry_MX_1.00u_Plate
- SW42: value ~ -> S; footprint JLClib:SW_Cherry_MX_1.00u_Plate -> Button_Switch_Keyboard:SW_Cherry_MX_1.00u_Plate
- SW43: value ~ -> D; footprint JLClib:SW_Cherry_MX_1.00u_Plate -> Button_Switch_Keyboard:SW_Cherry_MX_1.00u_Plate
- SW44: value ~ -> F; footprint JLClib:SW_Cherry_MX_1.00u_Plate -> Button_Switch_Keyboard:SW_Cherry_MX_1.00u_Plate
- SW45: value ~ -> G; footprint JLClib:SW_Cherry_MX_1.00u_Plate -> Button_Switch_Keyboard:SW_Cherry_MX_1.00u_Plate
- SW46: value ~ -> H; footprint JLClib:SW_Cherry_MX_1.00u_Plate -> Button_Switch_Keyboard:SW_Cherry_MX_1.00u_Plate
- SW47: value ~ -> J; footprint JLClib:SW_Cherry_MX_1.00u_Plate -> Button_Switch_Keyboard:SW_Cherry_MX_1.00u_Plate
- SW48: value ~ -> K; footprint JLClib:SW_Cherry_MX_1.00u_Plate -> Button_Switch_Keyboard:SW_Cherry_MX_1.00u_Plate
- SW49: value ~ -> L; footprint JLClib:SW_Cherry_MX_1.00u_Plate -> Button_Switch_Keyboard:SW_Cherry_MX_1.00u_Plate
- SW5: value ~ -> £ 3; footprint JLClib:SW_Cherry_MX_1.00u_Plate -> Button_Switch_Keyboard:SW_Cherry_MX_1.00u_Plate
- SW5: footprint JLClib:SW_Cherry_MX_1.00u_Plate -> Button_Switch_Keyboard:SW_Cherry_MX_1.00u_Plate
- SW50: value ~ -> : ;; footprint JLClib:SW_Cherry_MX_1.00u_Plate -> Button_Switch_Keyboard:SW_Cherry_MX_1.00u_Plate
- SW51: value ~ -> @ '; footprint JLClib:SW_Cherry_MX_1.00u_Plate -> Button_Switch_Keyboard:SW_Cherry_MX_1.00u_Plate
- SW52: value ~ -> ~ #; footprint JLClib:SW_Cherry_MX_1.00u_Plate -> Button_Switch_Keyboard:SW_Cherry_MX_1.00u_Plate
- SW53: value ~ -> 4 ←; footprint JLClib:SW_Cherry_MX_1.00u_Plate -> Button_Switch_Keyboard:SW_Cherry_MX_1.00u_Plate
- SW54: value ~ -> 5; footprint JLClib:SW_Cherry_MX_1.00u_Plate -> Button_Switch_Keyboard:SW_Cherry_MX_1.00u_Plate
- SW55: value ~ -> 6 →; footprint JLClib:SW_Cherry_MX_1.00u_Plate -> Button_Switch_Keyboard:SW_Cherry_MX_1.00u_Plate
- SW56: value ~ -> Shift; footprint JLClib:SW_Cherry_MX_1.00u_Plate -> Button_Switch_Keyboard:SW_Cherry_MX_1.25u_Plate
- SW57: value ~ -> | \; footprint JLClib:SW_Cherry_MX_1.00u_Plate -> Button_Switch_Keyboard:SW_Cherry_MX_1.00u_Plate
- SW58: value ~ -> Z; footprint JLClib:SW_Cherry_MX_1.00u_Plate -> Button_Switch_Keyboard:SW_Cherry_MX_1.00u_Plate
- SW59: value ~ -> X; footprint JLClib:SW_Cherry_MX_1.00u_Plate -> Button_Switch_Keyboard:SW_Cherry_MX_1.00u_Plate
- SW6: value ~ -> $ 4; footprint JLClib:SW_Cherry_MX_1.00u_Plate -> Button_Switch_Keyboard:SW_Cherry_MX_1.00u_Plate
- SW60: value ~ -> C; footprint JLClib:SW_Cherry_MX_1.00u_Plate -> Button_Switch_Keyboard:SW_Cherry_MX_1.00u_Plate
- SW61: value ~ -> V; footprint JLClib:SW_Cherry_MX_1.00u_Plate -> Button_Switch_Keyboard:SW_Cherry_MX_1.00u_Plate
- SW62: value ~ -> B; footprint JLClib:SW_Cherry_MX_1.00u_Plate -> Button_Switch_Keyboard:SW_Cherry_MX_1.00u_Plate
- SW63: value ~ -> N; footprint JLClib:SW_Cherry_MX_1.00u_Plate -> Button_Switch_Keyboard:SW_Cherry_MX_1.00u_Plate
- SW64: value ~ -> M; footprint JLClib:SW_Cherry_MX_1.00u_Plate -> Button_Switch_Keyboard:SW_Cherry_MX_1.00u_Plate
- SW65: value ~ -> < ,; footprint JLClib:SW_Cherry_MX_1.00u_Plate -> Button_Switch_Keyboard:SW_Cherry_MX_1.00u_Plate
- SW66: value ~ -> > .; footprint JLClib:SW_Cherry_MX_1.00u_Plate -> Button_Switch_Keyboard:SW_Cherry_MX_1.00u_Plate
- SW67: value ~ -> ? /; footprint JLClib:SW_Cherry_MX_1.00u_Plate -> Button_Switch_Keyboard:SW_Cherry_MX_1.00u_Plate
- SW69: renamed from SW68; value ~ -> ↑; footprint JLClib:SW_Cherry_MX_1.00u_Plate -> Button_Switch_Keyboard:SW_Cherry_MX_1.00u_Plate
- SW7: value ~ -> % 5; footprint JLClib:SW_Cherry_MX_1.00u_Plate -> Button_Switch_Keyboard:SW_Cherry_MX_1.00u_Plate
- SW70: renamed from SW69; value ~ -> 1 End; footprint JLClib:SW_Cherry_MX_1.00u_Plate -> Button_Switch_Keyboard:SW_Cherry_MX_1.00u_Plate
- SW71: renamed from SW70; value ~ -> 2 ↓; footprint JLClib:SW_Cherry_MX_1.00u_Plate -> Button_Switch_Keyboard:SW_Cherry_MX_1.00u_Plate
- SW72: renamed from SW71; value ~ -> 3 PgDn; footprint JLClib:SW_Cherry_MX_1.00u_Plate -> Button_Switch_Keyboard:SW_Cherry_MX_1.00u_Plate
- SW73: renamed from SW72; value ~ -> Enter; footprint JLClib:SW_Cherry_MX_1.00u_Plate -> Button_Switch_Keyboard:SW_Cherry_MX_2.00u_Vertical_Plate
- SW74: renamed from SW73; value ~ -> Ctrl; footprint JLClib:SW_Cherry_MX_1.00u_Plate -> Button_Switch_Keyboard:SW_Cherry_MX_1.25u_Plate
- SW75: renamed from SW74; value ~ -> Win; footprint JLClib:SW_Cherry_MX_1.00u_Plate -> Button_Switch_Keyboard:SW_Cherry_MX_1.25u_Plate
- SW76: renamed from SW75; value ~ -> Alt; footprint JLClib:SW_Cherry_MX_1.00u_Plate -> Button_Switch_Keyboard:SW_Cherry_MX_1.25u_Plate
- SW77: renamed from SW76; value ~ -> (none); footprint JLClib:SW_Cherry_MX_1.00u_Plate -> Button_Switch_Keyboard:SW_Cherry_MX_6.25u_Plate
- SW78: renamed from SW77; value ~ -> AltGr; footprint JLClib:SW_Cherry_MX_1.00u_Plate -> Button_Switch_Keyboard:SW_Cherry_MX_1.25u_Plate
- SW79: renamed from SW78; value ~ -> Fn; footprint JLClib:SW_Cherry_MX_1.00u_Plate -> Button_Switch_Keyboard:SW_Cherry_MX_1.25u_Plate
- SW8: value ~ -> ^ 6; footprint JLClib:SW_Cherry_MX_1.00u_Plate -> Button_Switch_Keyboard:SW_Cherry_MX_1.00u_Plate
- SW80: renamed from SW79; value ~ -> ←; footprint JLClib:SW_Cherry_MX_1.00u_Plate -> Button_Switch_Keyboard:SW_Cherry_MX_1.00u_Plate
- SW81: renamed from SW80; value ~ -> ↓; footprint JLClib:SW_Cherry_MX_1.00u_Plate -> Button_Switch_Keyboard:SW_Cherry_MX_1.00u_Plate
- SW82: renamed from SW81; value ~ -> →; footprint JLClib:SW_Cherry_MX_1.00u_Plate -> Button_Switch_Keyboard:SW_Cherry_MX_1.00u_Plate
- SW83: renamed from SW82; value ~ -> 0 Ins; footprint JLClib:SW_Cherry_MX_1.00u_Plate -> Button_Switch_Keyboard:SW_Cherry_MX_2.00u_Plate
- SW84: renamed from SW83; value ~ -> . Del; footprint JLClib:SW_Cherry_MX_1.00u_Plate -> Button_Switch_Keyboard:SW_Cherry_MX_1.00u_Plate
- SW9: value ~ -> & 7; footprint JLClib:SW_Cherry_MX_1.00u_Plate -> Button_Switch_Keyboard:SW_Cherry_MX_1.00u_Plate
- moved U20 413.0 mm to (361.9, 0.00)
- moved D20 405.3 mm to (362.0, 0.00)
- moved U39 402.5 mm to (361.9, 28.6)
- moved D39 397.6 mm to (362.0, 28.6)
- moved U17 394.2 mm to (304.8, 0.00)
- moved U19 394.0 mm to (342.9, 0.00)
- moved D1 388.2 mm to (-183.2, -95.6)
- moved U38 387.7 mm to (342.9, 19.1)
- moved D19 386.6 mm to (342.9, 0.00)
- moved D38 382.3 mm to (342.9, 19.1)
- moved U55 377.7 mm to (342.9, 38.1)
- moved U16 376.2 mm to (285.8, 0.00)
- moved U18 375.0 mm to (323.9, 0.00)
- moved K20 372.3 mm to (362.0, 0.00)
- moved D73 371.7 mm to (362.0, 66.7)
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- renumbered D68 to D69, D69 to D70, D70 to D71, D71 to D72, D72 to D73, D73 to D74, D74 to D75, D75 to D76, D76 to D77, D77 to D78, D78 to D79, D79 to D80, D80 to D81, D81 to D82, D82 to D83, D83 to D84, K59 to K56, K60 to K57, K61 to K58, K62 to K59, K63 to K60, K64 to K61, K65 to K62, K66 to K63, K67 to K64, K68 to K65, K69 to K66, K70 to K67, K71 to K68, K72 to K69, K73 to K70, K74 to K71, K75 to K72, K78 to K74, K79 to K75, K80 to K76, K81 to K77, K82 to K78, K83 to K79, K84 to K80, K85 to K81, K86 to K82, K87 to K83, K88 to K84, U73 to U74, U74 to U75, U75 to U76, U76 to U77, U77 to U78, U78 to U79, U79 to U80, U80 to U81, U81 to U82, U82 to U83, U83 to U84
Connections:
- U72 pad 4: Net-(U55-DOUT) -> Net-(U72-DIN)
Routing:
- net /Keyboard Matrix/Col1: track 57.0 -> 0.00 mm, vias 1 -> 0
- net /Keyboard Matrix/Col3: track 0.00 -> 57.0 mm, vias 0 -> 1
- net /Keyboard Matrix/Row0: track 37.3 -> 0.00 mm
- net /Keyboard Matrix/Col2: track 0.00 -> 37.3 mm
- net /Keyboard Matrix/Col0: track 34.3 -> 0.00 mm, vias 1 -> 0
- net /Keyboard Matrix/Col4: track 0.00 -> 34.3 mm, vias 0 -> 1
- net (no net): track 9.47 -> 0.00 mm
- net GND: track 39.7 -> 49.2 mm, vias 8 -> 9
- net /STM32/Boot: vias 1 -> 0
