File: leds.kicad_sch (KiCad schematic)
At the start: 9 parts, among them U3 A, U4 D, U5 S, U6 W

Commit message: Update Migouner2.kicad_pcb, Migouner2.kicad_prl, Migouner2.kicad_pro, and 4 more files
Parts:
- added K10, K11, K12, K13, K14, K15, K16, K17, K18, K19, K20, K21, K22, K23, K24, K25, K26, K27, K28, K29, K30, K31, K32, K33, K34, K35, K36, K37, K38, K39, K40, K41, K42, K43, K44, K45, K46, K47, K48, K49, K50, K51, K52, K53, K54, K55, K59, K6, K60, K61, K62, K63, K64, K65, K66, K67, K68, K69, K7, K70, K71, K72, K73, K74, K75, K78, K79, K8, K80, K81, K82, K83, K84, K85, K86, K87, K88, K9: 100nF, JLClib:C0402, symbol Device:C
- added U10, U11, U12, U13, U14, U15, U16, U17, U18, U19, U20, U21, U22, U23, U24, U25, U26, U27, U28, U29, U30, U31, U32, U33, U34, U35, U36, U37, U38, U39, U40, U41, U42, U43, U44, U45, U46, U47, U48, U49, U5, U50, U51, U52, U53, U54, U55, U56, U57, U58, U59, U60, U61, U62, U63, U64, U65, U66, U67, U68, U69, U7, U70, U71, U72, U73, U74, U75, U76, U77, U78, U79, U8, U80, U81, U82, U83, U9: ~, JLClib:LED-SMD_L3.2-W2.8-TR, symbol JLClib:SK6812MINI-E_C5149201
- U2: renamed from U3; value A -> ~
- U3: renamed from U5; value S -> ~
- U4: value D -> ~
- U6: value W -> ~
- renumbered C11 to K2, C12 to K3, C13 to K4, C14 to K5
Connections:
- net +5V: now also K10.1, K11.1, K12.1, K13.1, K14.1, K15.1, K16.1, K17.1, K18.1, K19.1, K20.1, K21.1, K22.1, K23.1, K24.1, K25.1, K26.1, K27.1, K28.1, K29.1, K30.1, K31.1, K32.1, K33.1, K34.1, K35.1, K36.1, K37.1, K38.1, K39.1, K40.1, K41.1, K42.1, K43.1, K44.1, K45.1, K46.1, K47.1, K48.1, K49.1, K50.1, K51.1, K52.1, K53.1, K54.1, K55.1, K59.1, K6.1, K60.1, K61.1, K62.1, K63.1, K64.1, K65.1, K66.1, K67.1, K68.1, K69.1, K7.1, K70.1, K71.1, K72.1, K73.1, K74.1, K75.1, K78.1, K79.1, K8.1, K80.1, K81.1, K82.1, K83.1, K84.1, K85.1, K86.1, K87.1, K88.1, K9.1, U73.1 (VDD), U74.1 (VDD), U75.1 (VDD), U76.1 (VDD), U77.1 (VDD), U78.1 (VDD), U79.1 (VDD), U80.1 (VDD), U81.1 (VDD), U82.1 (VDD), U83.1 (VDD); no longer U2.1 (VDD), U3.1 (VDD), U4.1 (VDD), U6.1 (VDD)
- net GND: now also K10.2, K11.2, K12.2, K13.2, K14.2, K15.2, K16.2, K17.2, K18.2, K19.2, K20.2, K21.2, K22.2, K23.2, K24.2, K25.2, K26.2, K27.2, K28.2, K29.2, K30.2, K31.2, K32.2, K33.2, K34.2, K35.2, K36.2, K37.2, K38.2, K39.2, K40.2, K41.2, K42.2, K43.2, K44.2, K45.2, K46.2, K47.2, K48.2, K49.2, K50.2, K51.2, K52.2, K53.2, K54.2, K55.2, K59.2, K6.2, K60.2, K61.2, K62.2, K63.2, K64.2, K65.2, K66.2, K67.2, K68.2, K69.2, K7.2, K70.2, K71.2, K72.2, K73.2, K74.2, K75.2, K78.2, K79.2, K8.2, K80.2, K81.2, K82.2, K83.2, K84.2, K85.2, K86.2, K87.2, K88.2, K9.2, U10.3 (GND), U11.3 (GND), U12.3 (GND), U13.3 (GND), U14.3 (GND), U15.3 (GND), U16.3 (GND), U17.3 (GND), U18.3 (GND), U19.3 (GND), U20.3 (GND), U5.3 (GND), U7.3 (GND), U8.3 (GND), U9.3 (GND)
- net at U6.4 (DIN): now also U5.2 (DOUT); no longer U3.2 (DOUT)
- net at U6.2 (DOUT): now also U7.4 (DIN); no longer U4.4 (DIN)
- net at U4.2 (DOUT): now also U5.4 (DIN)
- new net: U10.1 (VDD), U11.1 (VDD), U12.1 (VDD), U13.1 (VDD), U14.1 (VDD), U15.1 (VDD), U16.1 (VDD), U17.1 (VDD), U18.1 (VDD), U19.1 (VDD), U2.1 (VDD), U20.1 (VDD), U21.1 (VDD), U22.1 (VDD), U23.1 (VDD), U24.1 (VDD), U25.1 (VDD), U26.1 (VDD), U27.1 (VDD), U28.1 (VDD), U29.1 (VDD), U3.1 (VDD), U30.1 (VDD), U31.1 (VDD), U32.1 (VDD), U33.1 (VDD), U34.1 (VDD), U35.1 (VDD), U36.1 (VDD), U37.1 (VDD), U38.1 (VDD), U39.1 (VDD), U4.1 (VDD), U5.1 (VDD), U6.1 (VDD), U7.1 (VDD), U8.1 (VDD), U9.1 (VDD)
- new net: U32.4 (DIN), U33.2 (DOUT)
- new net: U21.3 (GND), U22.3 (GND), U23.3 (GND), U24.3 (GND), U25.3 (GND), U26.3 (GND), U27.3 (GND), U28.3 (GND), U29.3 (GND), U30.3 (GND), U31.3 (GND), U32.3 (GND), U33.3 (GND), U34.3 (GND), U35.3 (GND), U36.3 (GND), U37.3 (GND), U38.3 (GND), U39.3 (GND), U40.3 (GND), U41.3 (GND), U42.3 (GND), U43.3 (GND), U44.3 (GND), U45.3 (GND), U46.3 (GND), U47.3 (GND), U48.3 (GND), U49.3 (GND), U50.3 (GND), U51.3 (GND), U52.3 (GND), U53.3 (GND), U54.3 (GND), U55.3 (GND)
- new net: U33.4 (DIN), U34.2 (DOUT)
- new net: U28.4 (DIN), U29.2 (DOUT)
- new net: U29.4 (DIN), U30.2 (DOUT)
- new net: U73.2 (DOUT), U74.4 (DIN)
- new net: U56.3 (GND), U57.3 (GND), U58.3 (GND), U59.3 (GND), U60.3 (GND), U61.3 (GND), U62.3 (GND), U63.3 (GND), U64.3 (GND), U65.3 (GND), U66.3 (GND), U67.3 (GND), U68.3 (GND), U69.3 (GND), U70.3 (GND), U71.3 (GND), U72.3 (GND), U73.3 (GND), U74.3 (GND), U75.3 (GND), U76.3 (GND), U77.3 (GND), U78.3 (GND), U79.3 (GND), U80.3 (GND), U81.3 (GND), U82.3 (GND), U83.3 (GND)
- new net: U56.2 (DOUT), U73.4 (DIN)
- new net: U40.1 (VDD), U41.1 (VDD), U42.1 (VDD), U43.1 (VDD), U44.1 (VDD), U45.1 (VDD), U46.1 (VDD), U47.1 (VDD), U48.1 (VDD), U49.1 (VDD), U50.1 (VDD), U51.1 (VDD), U53.1 (VDD), U54.1 (VDD), U55.1 (VDD), U56.1 (VDD), U57.1 (VDD), U58.1 (VDD), U59.1 (VDD), U60.1 (VDD), U61.1 (VDD), U62.1 (VDD), U63.1 (VDD), U64.1 (VDD), U65.1 (VDD), U66.1 (VDD), U67.1 (VDD), U68.1 (VDD), U69.1 (VDD), U70.1 (VDD), U71.1 (VDD), U72.1 (VDD)
- new net: U69.4 (DIN), U70.2 (DOUT)
- new net: U70.4 (DIN), U71.2 (DOUT)
- new net: U47.2 (DOUT), U48.4 (DIN)
- new net: U46.2 (DOUT), U47.4 (DIN)
- new net: U40.2 (DOUT), U41.4 (DIN)
- new net: U21.2 (DOUT), U40.4 (DIN)
- new net: U24.4 (DIN), U25.2 (DOUT)
- new net: U25.4 (DIN), U26.2 (DOUT)
- new net: U67.4 (DIN), U68.2 (DOUT)
- new net: U68.4 (DIN), U69.2 (DOUT)
- new net: U53.2 (DOUT), U54.4 (DIN)
- new net: U52.2 (DOUT), U53.4 (DIN)
- new net: U82.2 (DOUT), U83.4 (DIN)
- new net: U27.4 (DIN), U28.2 (DOUT)
- new net: U51.2 (DOUT), U52.4 (DIN)
- new net: U50.2 (DOUT), U51.4 (DIN)
- new net: U8.2 (DOUT), U9.4 (DIN)
- new net: U7.2 (DOUT), U8.4 (DIN)
- new net: U61.4 (DIN), U62.2 (DOUT)
- new net: U62.4 (DIN), U63.2 (DOUT)
- new net: U30.4 (DIN), U31.2 (DOUT)
- new net: U31.4 (DIN), U32.2 (DOUT)
- new net: U55.2 (DOUT), U72.4 (DIN)
- new net: U54.2 (DOUT), U55.4 (DIN)
- new net: U35.4 (DIN), U36.2 (DOUT)
- new net: U36.4 (DIN), U37.2 (DOUT)
- new net: U17.2 (DOUT), U18.4 (DIN)
- new net: U16.2 (DOUT), U17.4 (DIN)
- new net: U42.2 (DOUT), U43.4 (DIN)
- new net: U41.2 (DOUT), U42.4 (DIN)
- new net: U57.4 (DIN), U58.2 (DOUT)
- new net: U58.4 (DIN), U59.2 (DOUT)
- new net: U49.2 (DOUT), U50.4 (DIN)
- new net: U48.2 (DOUT), U49.4 (DIN)
- new net: U44.2 (DOUT), U45.4 (DIN)
- new net: U43.2 (DOUT), U44.4 (DIN)
- new net: U14.2 (DOUT), U15.4 (DIN)
- new net: U13.2 (DOUT), U14.4 (DIN)
- new net: U18.2 (DOUT), U19.4 (DIN)
- new net: U15.2 (DOUT), U16.4 (DIN)
- new net: U3.2 (DOUT), U4.4 (DIN)
- new net: U37.4 (DIN), U38.2 (DOUT)
- new net: U38.4 (DIN), U39.2 (DOUT)
- new net: U10.2 (DOUT), U11.4 (DIN)
- new net: U10.4 (DIN), U9.2 (DOUT)
- new net: U63.4 (DIN), U64.2 (DOUT)
- new net: U34.4 (DIN), U35.2 (DOUT)
- new net: U81.2 (DOUT), U82.4 (DIN)
- new net: U64.4 (DIN), U65.2 (DOUT)
- new net: U65.4 (DIN), U66.2 (DOUT)
- new net: U45.2 (DOUT), U46.4 (DIN)
- new net: U26.4 (DIN), U27.2 (DOUT)
- new net: U23.4 (DIN), U24.2 (DOUT)
- new net: U71.4 (DIN), U72.2 (DOUT)
- new net: U12.2 (DOUT), U13.4 (DIN)
- new net: U11.2 (DOUT), U12.4 (DIN)
- new net: U22.4 (DIN), U23.2 (DOUT)
- new net: U19.2 (DOUT), U20.4 (DIN)
- new net: U20.2 (DOUT), U39.4 (DIN)
- new net: U79.2 (DOUT), U80.4 (DIN)
- new net: U78.2 (DOUT), U79.4 (DIN)
- new net: U77.2 (DOUT), U78.4 (DIN)
- new net: U76.2 (DOUT), U77.4 (DIN)
- new net: U66.4 (DIN), U67.2 (DOUT)
- new net: U80.2 (DOUT), U81.4 (DIN)
- new net: U21.4 (DIN), U22.2 (DOUT)
- new net: U56.4 (DIN), U57.2 (DOUT)
- new net: U60.4 (DIN), U61.2 (DOUT)
- new net: U74.2 (DOUT), U75.4 (DIN)
- new net: U59.4 (DIN), U60.2 (DOUT)
- new net: U75.2 (DOUT), U76.4 (DIN)
Other:
- moved on the sheet: K2, K3, K4, K5, R2, U2, U3

Commit message: Board scripting
Parts:
- added K73: 100nF, JLClib:C0402, symbol Device:C
- added U73: ~, JLClib:LED-SMD_L3.2-W2.8-TR, symbol JLClib:SK6812MINI-E_C5149201
- renumbered K59 to K56, K60 to K57, K61 to K58, K62 to K59, K63 to K60, K64 to K61, K65 to K62, K66 to K63, K67 to K64, K68 to K65, K69 to K66, K70 to K67, K71 to K68, K72 to K69, K73 to K70, K74 to K71, K75 to K72, K78 to K74, K79 to K75, K80 to K76, K81 to K77, K82 to K78, K83 to K79, K84 to K80, K85 to K81, K86 to K82, K87 to K83, K88 to K84, U73 to U74, U74 to U75, U75 to U76, U76 to U77, U77 to U78, U78 to U79, U79 to U80, U80 to U81, U81 to U82, U82 to U83, U83 to U84
Connections:
- net +5V: now also K73.1
- net GND: now also K73.2
- net at U56.3 (GND), U57.3 (GND), U58.3 (GND)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: now also U73.3 (GND)
- net at U40.1 (VDD), U41.1 (VDD), U42.1 (VDD)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: now also U73.1 (VDD)
- net at U55.2 (DOUT): now also U73.4 (DIN); no longer U72.4 (DIN)
- new net: U72.4 (DIN), U73.2 (DOUT)
